File: nasa-badge.kicad_pcb (KiCad board)
At the start: 2 copper layers, 99.7 x 81.6 mm, 60 parts, among them J1 USB_C_Receptacle_USB2.0, J2 Conn_01x04_Female, Q1 PZT3904, Q2 PZT3904, Q3 PZT3904, SW1 SW_Push, SW2 SW_Push, U1 MCP73831-2-OT, U2 AMS1117-3.3, U3 FT232RL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

Commit message: rev 0.2
Parts:
- removed the G*** at (147.3, 90.8) (x2)
- added G*** (x2): LOGO, LOGO, F.Cu at (147.3, 90.8)
- C3, C5: value 100uF -> optional
- R2, R3: value 56k -> 51k
- R4, R5, R6: value 1.5K -> 1.8K
- U2: value AMS1117-3.3 -> AP2114H-3.3
