File: nasa-badge.sch (KiCad schematic (older format))
At the start: 54 parts, among them J1 USB_C_Receptacle_USB2.0, J2 Conn_01x04_Female, Q1 PZT3904, Q2 PZT3904, Q3 PZT3904, SW1 SW_Push, SW2 SW_Push, U1 MCP73831-2-OT, U2 AMS1117-3.3, U3 FT232RL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

Commit message: rev 0.2
Parts:
- removed U2: AMS1117-3.3, Package_TO_SOT_SMD:SOT-223-3_TabPin2, symbol Regulator_Linear:AMS1117-3.3
- added U2: AP2114H-3.3, Package_TO_SOT_SMD:SOT-223-3_TabPin2, symbol custom:AP2114H-3.3
- C3, C5: value 100uF -> optional
- R2, R3: value 56k -> 51k
- R4, R5, R6: value 1.5K -> 1.8K
Connections:
- net +3V3: now also U2.2 (VO)
- net GND: now also U2.1 (ADJ)
- net at BT1.1 (+), C2.1, C3.1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: now also U2.3 (VI)
Other:
- note removed: "Ggf widerstand. Siehe FTDI-Datasheet"
Changed lines of the file:
@@
 Title ""
 Date ""
-Rev ""
+Rev "0.2"
 Comp ""
 Comment1 ""
@@
 P 2750 1450
 F 0 "R3" V 2543 1450 50  0000 C CNN
-F 1 "56k" V 2634 1450 50  0000 C CNN
+F 1 "51k" V 2634 1450 50  0000 C CNN
 F 2 "Resistor_SMD:R_0805_2012Metric_Pad1.15x1.40mm_HandSolder" V 2680 1450 50  0001 C CNN
 F 3 "~" H 2750 1450 50  0001 C CNN
@@
 P 2500 1350
 F 0 "R2" V 2293 1350 50  0000 C CNN
-F 1 "56k" V 2384 1350 50  0000 C CNN
+F 1 "51k" V 2384 1350 50  0000 C CNN
 F 2 "Resistor_SMD:R_0805_2012Metric_Pad1.15x1.40mm_HandSolder" V 2430 1350 50  0001 C CNN
 F 3 "~" H 2500 1350 50  0001 C CNN
@@
 Wire Wire Line
 	2300 1950 2300 1900
-Text Notes 350  2700 0    50   ~ 0
-Ggf widerstand. Siehe FTDI-Datasheet
 $Comp
 L power:GND #PWR0104
@@
 	1    0    0    -1
 $EndComp
-$Comp
-L Regulator_Linear:AMS1117-3.3 U2
-U 1 1 5F1B5E0F
-P 4450 4250
-F 0 "U2" H 4450 4492 50  0000 C CNN
-F 1 "AMS1117-3.3" H 4450 4401 50  0000 C CNN
-F 2 "Package_TO_SOT_SMD:SOT-223-3_TabPin2" H 4450 4450 50  0001 C CNN
-F 3 "http://www.advanced-monolithic.com/pdf/ds1117.pdf" H 4550 4000 50  0001 C CNN
-	1    4450 4250
-	1    0    0    -1
-$EndComp
 Wire Wire Line
 	3300 4650 3300 4250
@@
 P 3850 4400
 F 0 "C3" H 3965 4446 50  0000 L CNN
-F 1 "100uF" H 3965 4355 50  0000 L CNN
+F 1 "optional" H 3965 4355 50  0000 L CNN
 F 2 "Capacitor_SMD:C_0805_2012Metric_Pad1.15x1.40mm_HandSolder" H 3888 4250 50  0001 C CNN
 F 3 "~" H 3850 4400 50  0001 C CNN
@@
 P 5300 4400
 F 0 "C5" H 5415 4446 50  0000 L CNN
-F 1 "100uF" H 5415 4355 50  0000 L CNN
+F 1 "optional" H 5415 4355 50  0000 L CNN
 F 2 "Capacitor_SMD:C_0805_2012Metric_Pad1.15x1.40mm_HandSolder" H 5338 4250 50  0001 C CNN
 F 3 "~" H 5300 4400 50  0001 C CNN
@@
 	1    0    0    -1
 $EndComp
-Wire Wire Line
-	4450 4550 4450 4650
 $Comp
 L power:+3V3 #PWR0114
@@
 P 8600 2350
 F 0 "R4" V 8807 2350 50  0000 C CNN
-F 1 "1.5K" V 8716 2350 50  0000 C CNN
+F 1 "1.8K" V 8716 2350 50  0000 C CNN
 F 2 "Resistor_SMD:R_0805_2012Metric_Pad1.15x1.40mm_HandSolder" V 8530 2350 50  0001 C CNN
 F 3 "~" H 8600 2350 50  0001 C CNN
@@
 P 8600 3800
 F 0 "R5" V 8807 3800 50  0000 C CNN
-F 1 "1.5K" V 8716 3800 50  0000 C CNN
+F 1 "1.8K" V 8716 3800 50  0000 C CNN
 F 2 "Resistor_SMD:R_0805_2012Metric_Pad1.15x1.40mm_HandSolder" V 8530 3800 50  0001 C CNN
 F 3 "~" H 8600 3800 50  0001 C CNN
@@
 P 8600 5250
 F 0 "R6" V 8807 5250 50  0000 C CNN
-F 1 "1.5K" V 8716 5250 50  0000 C CNN
+F 1 "1.8K" V 8716 5250 50  0000 C CNN
 F 2 "Resistor_SMD:R_0805_2012Metric_Pad1.15x1.40mm_HandSolder" V 8530 5250 50  0001 C CNN
 F 3 "~" H 8600 5250 50  0001 C CNN
@@
 Wire Wire Line
 	6700 1950 6750 1950
+Wire Wire Line
+	4450 4550 4450 4650
+$Comp
+L custom:AP2114H-3.3 U2
+U 1 1 5F41B879
+P 4450 4250
+F 0 "U2" H 4450 4492 50  0000 C CNN
+F 1 "AP2114H-3.3" H 4450 4401 50  0000 C CNN
+F 2 "Package_TO_SOT_SMD:SOT-223-3_TabPin2" H 4450 4450 50  0001 C CNN
+F 3 "http://www.diodes.com/datasheets/AP1117.pdf" H 4550 4000 50  0001 C CNN
+	1    4450 4250
+	1    0    0    -1
+$EndComp
 $EndSCHEMATC
