File: hardware/nasa-badge.kicad_pcb (KiCad board)
At the start: 2 copper layers, 99.7 x 81.6 mm, 60 parts, among them J1 USB_C_Receptacle_USB2.0, J2 Conn_01x04_Female, Q1 PZT3904, Q2 PZT3904, Q3 PZT3904, SW1 SW_Push, SW2 SW_Push, U1 MCP73831-2-OT, U2 AP2114H-3.3, U3 FT232RL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

Commit message: add board version number
Parts:
- removed the G*** at (147.3, 90.8) (x2)
- added G*** (x2): LOGO, LOGO, F.Cu at (147.3, 90.8)
Changed lines of the file:
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@@
   )
   (page A4)
+  (title_block
+    (rev 0.2)
+  )
   (layers
     (0 F.Cu signal)
